File: Encoders/PCB/quadrature_decoder/board.sch (EAGLE design)
At the start: 14 parts

Commit message: new board layout
Parts:
- renumbered SV1 to CON2, SV2 to UART, SV3 to CON3, SV4 to CON1, SV5 to CON5, SV6 to CON6, SV7 to CON4, U$1 to IC3, U$2 to IC1, U$3 to IC5, U$4 to IC6, U$5 to IC4, U$6 to IC2

Commit message: new board
Connections:
- removed net N$1: CON2.1, IC2.VSS
- removed net N$11: CON1.1, IC1.VSS
- removed net N$15: CON5.1, IC5.VSS
- removed net N$19: CON6.1, IC6.VSS
- removed net N$23: CON4.1, IC4.VSS
- removed net N$6: CON3.1, IC3.VSS
- net 5V: now also U$7.5V
- net GND: now also CON1.1, CON2.1, CON3.1, CON4.1, CON5.1, CON6.1, IC1.VSS, IC2.VSS, IC3.VSS, IC4.VSS, IC5.VSS, IC6.VSS
